File: lumberjack.kicad_sch (KiCad schematic)
At the start: 159 parts, among them J1 USB, J2 AVR_ISP_6, J3 JST, J4 JST, SW1 RESET, SW2 BOOT, U1 ATMEGA328-PU, Y1 16MHz

Commit message: 修改丝印，增加屏幕插座
Parts:
- removed LED1: RED, LED_THT:LED_D3.0mm, symbol Device:LED_Small
- removed LED2: GREEN, LED_THT:LED_D3.0mm, symbol Device:LED_Small
- removed R7, R8: 1.5k, Resistor_THT:R_Axial_DIN0204_L3.6mm_D1.6mm_P7.62mm_Horizontal, symbol Device:R_Small
- added J5: Conn_01x04_Female, Connector_PinHeader_2.54mm:PinHeader_1x04_P2.54mm_Vertical, symbol Connector:Conn_01x04_Female
Connections:
- net +5V: now also J5.2 (Pin_2)
- net GND: now also J5.1 (Pin_1)
- net LED1 renamed SCL
- net SCL: now also J5.3 (Pin_3)
- net LED2 renamed SDA
- net SDA: now also J5.4 (Pin_4)

Commit message: 更改了led，增加oled屏幕
Parts:
- U1: footprint Package_DIP:DIP-28_W7.62mm -> Package_DIP:DIP-28_W7.62mm_Socket
Changed lines of the file:
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@@
     (property "Reference" "U1" (id 0) (at 50.8 140.97 0))
     (property "Value" "ATMEGA328-PU" (id 1) (at 50.8 143.51 0))
-    (property "Footprint" "Package_DIP:DIP-28_W7.62mm" (id 2) (at 50.8 142.24 0)
+    (property "Footprint" "Package_DIP:DIP-28_W7.62mm_Socket" (id 2) (at 50.8 142.24 0)
       (effects (font (size 1.27 1.27) italic) hide)
     )
@@
     )
     (path "/00000000-0000-0000-0000-00005c16fb14"
-      (reference "U1") (unit 1) (value "ATMEGA328-PU") (footprint "Package_DIP:DIP-28_W7.62mm")
+      (reference "U1") (unit 1) (value "ATMEGA328-PU") (footprint "Package_DIP:DIP-28_W7.62mm_Socket")
     )
     (path "/00000000-0000-0000-0000-00005c3232f3"
